File: W5500-POE-Ethernet-SPI-breackout/W5500-POE-Ethernet-SPI-breackout.kicad_sch (KiCad schematic)
At the start: 66 parts, among them IC1 AP2112M-3.3TRG1, J1 ARJM11C7-114-BA-EW2, J2 Conn_02x04_Odd_Even, J3 Conn_01x08, J4 Conn_01x02, U1 W5500, Y1 Crystal 25MHz

Commit message: f
Parts:
- C1, C10, C11, C12, C13, C14, C15, C16, C17, C18, C2, C3, C4, C5, C6, C7, C8, C9: footprint (none) -> Capacitor_SMD:C_0805_2012Metric
- FID1, FID2, FID3, FID4, FID5: now left out of the parts list
- FID6: value (none) -> Fiducial; footprint (none) -> Symbol:WEEE-Logo_5.6x8mm_SilkScreen; now left out of the parts list
- IC1: footprint SamacSys_Parts:SOIC127P600X170-8N -> SOIC127P600X170-8N
- J1: footprint SamacSys_Parts:ARJM11C7114BAEW2 -> ARJM11C7114BAEW2
Other:
- moved on the sheet: C1, C11, C12, C13, C14, C15, C18, C2, C3, C4, C5, C6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
