File: W5500-POE-Ethernet-SPI-breackout/W5500-POE-Ethernet-SPI-breackout.kicad_pcb (KiCad board)
At the start: 2 copper layers, 70.2 x 33 mm, 78 parts, among them IC1 AP2112M-3.3TRG1, J1 ARJM11C7-114-BA-EW2, J2 Conn_02x04_Odd_Even, J3 Conn_01x08, J4 Conn_01x02, U1 W5500, Y1 Crystal 25MHz

Commit message: e
Parts:
- added  : LOGO, LOGO, B.Cu at (191.8, 78.0)
Routing:
- net +3.3VA: track 53.2 -> 56.8 mm
- net +3V3: track 89.5 -> 88.9 mm

Commit message: f
Parts:
- moved kibuzzard-6280C015 1.35 mm to (178.8, 62.4)
- moved kibuzzard-62827A52 0.66 mm to (180.9, 88.4)
Other:
- board size 70.2 x 33 mm -> 70.3 x 33 mm

Commit message: f
Changed lines of the file:
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@@
     (property "Sheetfile" "W5500-POE-Ethernet-SPI-breackout.kicad_sch")
     (property "Sheetname" "")
-    (attr smd)
+    (property "exclude_from_bom" "")
+    (attr smd exclude_from_bom)
     (fp_text reference "FID1" (at -2.413 0) (layer "F.SilkS")
       (effects (font (size 1 1) (thickness 0.15)))
@@
     (property "Sheetfile" "W5500-POE-Ethernet-SPI-breackout.kicad_sch")
     (property "Sheetname" "")
-    (attr smd)
+    (property "exclude_from_bom" "")
+    (attr smd exclude_from_bom)
     (fp_text reference "FID2" (at 0 -1.5 90) (layer "F.SilkS")
       (effects (font (size 1 1) (thickness 0.15)))
@@
     (property "Sheetname" "")
     (attr through_hole)
-    (fp_text reference "J1" (at 4.2164 13.6652 90) (layer "F.SilkS")
+    (fp_text reference "J1" (at -5.715 9.04 90) (layer "F.SilkS")
       (effects (font (size 1.27 1.27) (thickness 0.254)))
     )
@@
       (effects (font (size 1.27 1.27) (thickness 0.254)))
     )
+    (fp_line (start 2.235 -1.61) (end 2.235 4) (layer "F.SilkS") (width 0.1))
     (fp_line (start -13.665 7.5) (end -13.665 19.69) (layer "F.SilkS") (width 0.1))
-    (fp_line (start -13.665 -1.5) (end -13.665 -1.61) (layer "F.SilkS") (width 0.1))
+    (fp_line (start -13.665 4) (end -13.665 -1.5) (layer "F.SilkS") (width 0.1))
+    (fp_line (start 0 -2.2) (end 0 -2.2) (layer "F.SilkS") (width 0.2))
     (fp_line (start -13.665 19.69) (end 2.235 19.69) (layer "F.SilkS") (width 0.1))
-    (fp_line (start 2.235 -1.61) (end 2.235 4) (layer "F.SilkS") (width 0.1))
-    (fp_line (start 2.235 19.69) (end 2.235 7.5) (layer "F.SilkS") (width 0.1))
     (fp_line (start 2.16 -1.61) (end 2.235 -1.61) (layer "F.SilkS") (width 0.1))
+    (fp_line (start -13.665 -1.5) (end -13.665 -1.61) (layer "F.SilkS") (width 0.1))
     (fp_line (start 0 -2) (end 0 -2) (layer "F.SilkS") (width 0.2))
-    (fp_line (start 0 -2.2) (end 0 -2.2) (layer "F.SilkS") (width 0.2))
+    (fp_line (start 2.235 19.69) (end 2.235 7.5) (layer "F.SilkS") (width 0.1))
     (fp_line (start -13.665 -1.61) (end 2.16 -1.61) (layer "F.SilkS") (width 0.1))
-    (fp_line (start -13.665 4) (end -13.665 -1.5) (layer "F.SilkS") (width 0.1))
-    (fp_arc (start 0 -2.2) (mid 0.1 -2.1) (end 0 -2) (layer "F.SilkS") (width 0.2))
     (fp_arc (start 0 -2) (mid -0.1 -2.1) (end 0 -2.2) (layer "F.SilkS") (width 0.2))
-    (fp_line (start 4.337 -2.61) (end 4.337 20.69) (layer "F.CrtYd") (width 0.1))
-    (fp_line (start -15.768 -2.61) (end 4.337 -2.61) (layer "F.CrtYd") (width 0.1))
+    (fp_arc (start 0 -2.2) (mid 0.1 -2.1) (end 0 -2) (layer "F.SilkS") (width 0.2))
     (fp_line (start 4.337 20.69) (end -15.768 20.69) (layer "F.CrtYd") (width 0.1))
+    (fp_line (start -15.768 -2.61) (end 4.337 -2.61) (layer "F.CrtYd") (width 0.1))
+    (fp_line (start 4.337 -2.61) (end 4.337 20.69) (layer "F.CrtYd") (width 0.1))
     (fp_line (start -15.768 20.69) (end -15.768 -2.61) (layer "F.CrtYd") (width 0.1))
+    (fp_line (start 2.235 19.69) (end -13.665 19.69) (layer "F.Fab") (width 0.2))
+    (fp_line (start -13.665 19.69) (end -13.665 -1.61) (layer "F.Fab") (width 0.2))
     (fp_line (start -13.665 -1.61) (end 2.235 -1.61) (layer "F.Fab") (width 0.2))
     (fp_line (start 2.235 -1.61) (end 2.235 19.69) (layer "F.Fab") (width 0.2))
-    (fp_line (start -13.665 19.69) (end -13.665 -1.61) (layer "F.Fab") (width 0.2))
-    (fp_line (start 2.235 19.69) (end -13.665 19.69) (layer "F.Fab") (width 0.2))
     (pad "" np_thru_hole circle locked (at 0 8.89 90) (size 3.25 3.25) (drill 3.25) (layers *.Cu *.Mask))
     (pad "" np_thru_hole circle locked (at -11.43 8.89 90) (size 3.25 3.25) (drill 3.25) (layers *.Cu *.Mask))
@@
     (property "Sheetname" "")
     (attr smd)
-    (fp_text reference "IC1" (at -0.127 -0.127 90) (layer "F.SilkS")
+    (fp_text reference "IC1" (at 0 0 180) (layer "F.SilkS")
       (effects (font (size 1.27 1.27) (thickness 0.254)))
     )
-    (fp_text value "AP2112M-3.3TRG1" (at 0 0) (layer "F.SilkS") hide
+    (fp_text value "AP2112M-3.3TRG1" (at 0 0 180) (layer "F.SilkS") hide
       (effects (font (size 1.27 1.27) (thickness 0.254)))
     )
-    (fp_text user "${REFERENCE}" (at 0 0) (layer "F.Fab")
+    (fp_text user "${REFERENCE}" (at 0 0 180) (layer "F.Fab")
       (effects (font (size 1.27 1.27) (thickness 0.254)))
     )
     (fp_line (start -3.45 -2.58) (end -1.95 -2.58) (layer "F.SilkS") (width 0.2))
-    (fp_line (start -1.6 2.45) (end -1.6 -2.45) (layer "F.SilkS") (width 0.2))
+    (fp_line (start -1.6 -2.45) (end 1.6 -2.45) (layer "F.SilkS") (width 0.2))
     (fp_line (start 1.6 -2.45) (end 1.6 2.45) (layer "F.SilkS") (width 0.2))
     (fp_line (start 1.6 2.45) (end -1.6 2.45) (layer "F.SilkS") (width 0.2))
-    (fp_line (start -1.6 -2.45) (end 1.6 -2.45) (layer "F.SilkS") (width 0.2))
+    (fp_line (start -1.6 2.45) (end -1.6 -2.45) (layer "F.SilkS") (width 0.2))
     (fp_line (start 3.7 -2.725) (end 3.7 2.725) (layer "F.CrtYd") (width 0.05))
     (fp_line (start -3.7 2.725) (end -3.7 -2.725) (layer "F.CrtYd") (width 0.05))
-    (fp_line (start -3.7 -2.725) (end 3.7 -2.725) (layer "F.CrtYd") (width 0.05))
     (fp_line (start 3.7 2.725) (end -3.7 2.725) (layer "F.CrtYd") (width 0.05))
-    (fp_line (start 1.95 2.45) (end -1.95 2.45) (layer "F.Fab") (width 0.1))
+    (fp_line (start -3.7 -2.725) (end 3.7 -2.725) (layer "F.CrtYd") (width 0.05))
     (fp_line (start -1.95 2.45) (end -1.95 -2.45) (layer "F.Fab") (width 0.1))
     (fp_line (start -1.95 -2.45) (end 1.95 -2.45) (layer "F.Fab") (width 0.1))
     (fp_line (start 1.95 -2.45) (end 1.95 2.45) (layer "F.Fab") (width 0.1))
     (fp_line (start -1.95 -1.18) (end -0.68 -2.45) (layer "F.Fab") (width 0.1))
+    (fp_line (start 1.95 2.45) (end -1.95 2.45) (layer "F.Fab") (width 0.1))
     (pad "1" smd rect locked (at -2.7 -1.905 270) (size 0.65 1.5) (layers "F.Cu" "F.Paste" "F.Mask")
       (net 3 "+3V3") (pinfunction "VOUT") (pintype "passive"))
@@
     (property "Sheetfile" "W5500-POE-Ethernet-SPI-breackout.kicad_sch")
     (property "Sheetname" "")
-    (attr exclude_from_pos_files)
+    (property "exclude_from_bom" "")
+    (attr exclude_from_pos_files exclude_from_bom)
     (fp_text reference "FID6" (at 0 0) (layer "B.SilkS") hide
       (effects (font (size 1 1) (thickness 0.15)) (justify mirror))
@@
     (property "Sheetfile" "W5500-POE-Ethernet-SPI-breackout.kicad_sch")
     (property "Sheetname" "")
-    (attr exclude_from_pos_files)
+    (property "exclude_from_bom" "")
+    (attr exclude_from_pos_files exclude_from_bom)
     (fp_text reference "FID5" (at 0 0 90) (layer "B.SilkS") hide
       (effects (font (size 1 1) (thickness 0.15)) (justify mirror))
@@
     (property "Sheetfile" "W5500-POE-Ethernet-SPI-breackout.kicad_sch")
     (property "Sheetname" "")
-    (attr exclude_from_pos_files)
+    (property "exclude_from_bom" "")
+    (attr exclude_from_pos_files exclude_from_bom)
     (fp_text reference "FID3" (at 0 8.89) (layer "B.SilkS") hide
       (effects (font (size 1 1) (thickness 0.15)) (justify mirror))
@@
     (property "Sheetfile" "W5500-POE-Ethernet-SPI-breackout.kicad_sch")
     (property "Sheetname" "")
-    (attr exclude_from_pos_files)
+    (property "exclude_from_bom" "")
+    (attr exclude_from_pos_files exclude_from_bom)
     (fp_text reference "FID4" (at 0.762 4.191) (layer "F.Fab")
       (effects (font (size 1.524 1.524) (thickness 0.15)) (justify mirror))
@@
     )
   )
+  (zone (net 36) (net_name "/W5500_RST") (layer "F.Cu") (hatch edge 0.508)
+    (priority 16962)
+    (connect_pads yes (clearance 0))
+    (min_thickness 0.0254) (filled_areas_thickness no)
+    (fill yes (thermal_gap 0.508) (thermal_bridge_width 0.508))
+    (polygon
+      (pts
+        (xy 186.575002 88.354225)
+        (xy 186.513346 88.287949)
+        (xy 186.466415 88.227737)
+        (xy 186.431583 88.171824)
+        (xy 186.406222 88.118449)
+        (xy 186.387706 88.065846)
+        (xy 186.373407 88.012254)
+        (xy 186.360699 87.95591)
+        (xy 186.346953 87.89505)
+        (xy 186.329545 87.827911)
+        (xy 186.305846 87.75273)
+        (xy 185.786579 87.742579)
+        (xy 185.79673 88.261846)
+        (xy 185.871911 88.285545)
+        (xy 185.93905 88.302953)
+        (xy 185.99991 88.316699)
+        (xy 186.056254 88.329407)
+        (xy 186.109846 88.343706)
+        (xy 186.162449 88.362222)
+        (xy 186.215824 88.387583)
+        (xy 186.271737 88.422415)
+        (xy 186.331949 88.469346)
+        (xy 186.398225 88.531002)
+      )
+    )
+  )
   (zone (net 3) (net_name "+3V3") (layer "F.Cu") (hatch edge 0.508)
     (priority 16962)
@@
       )
     )
-  )
-  (zone (net 36) (net_name "/W5500_RST") (layer "F.Cu") (hatch edge 0.508)
-    (priority 16962)
-    (connect_pads yes (clearance 0))
-    (min_thickness 0.0254) (filled_areas_thickness no)
-    (fill yes (thermal_gap 0.508) (thermal_bridge_width 0.508))
-    (polygon
-      (pts
-        (xy 186.575002 88.354225)
-        (xy 186.513346 88.287949)
-        (xy 186.466415 88.227737)
-        (xy 186.431583 88.171824)
-        (xy 186.406222 88.118449)
-        (xy 186.387706 88.065846)
-        (xy 186.373407 88.012254)
-        (xy 186.360699 87.95591)
-        (xy 186.346953 87.89505)
-        (xy 186.329545 87.827911)
-        (xy 186.305846 87.75273)
-        (xy 185.786579 87.742579)
-        (xy 185.79673 88.261846)
-        (xy 185.871911 88.285545)
-        (xy 185.93905 88.302953)
-        (xy 185.99991 88.316699)
-        (xy 186.056254 88.329407)
-        (xy 186.109846 88.343706)
-        (xy 186.162449 88.362222)
-        (xy 186.215824 88.387583)
-        (xy 186.271737 88.422415)
-        (xy 186.331949 88.469346)
-        (xy 186.398225 88.531002)
-      )
-    )

Commit message: gg
Parts:
- added kibuzzard-6338560E: G***, kibuzzard-6338560E, B.Cu at (185.9, 84.7)
- added kibuzzard-63385628: G***, kibuzzard-63385628, B.Cu at (184.8, 82.1)
- added kibuzzard-63385636: G***, kibuzzard-63385636, B.Cu at (184.7, 79.6)
- added kibuzzard-6338564E: G***, kibuzzard-6338564E, B.Cu at (184.7, 77.1)
- added kibuzzard-6338565D: G***, kibuzzard-6338565D, B.Cu at (183.6, 74.4)
- added kibuzzard-6338566D: G***, kibuzzard-6338566D, B.Cu at (184.3, 72.0)
- added kibuzzard-6338567A: G***, kibuzzard-6338567A, B.Cu at (184.2, 69.5)
- added kibuzzard-63385685: G***, kibuzzard-63385685, B.Cu at (183.6, 66.7)
- moved   1.74 mm to (193.5, 78.2)
Routing:
- net GND: track 102.4 -> 106.9 mm, vias 62 -> 92
- net /act_led: track 54.6 -> 55.2 mm
